Commit message: errors on urdf and new softhand_plugins adaptation

File: franka_softhand_description/robot/franka_softhand.xacro (robot description, xacro)
@@ -5,7 +5,7 @@
     <!-- Should a franka_gripper be mounted at the flange?" -->
     <xacro:arg name="hand" default="false" />
-    <!-- Positional offset between $(arm_id)_hand -> $(arm_id)_hand_tcp [m]. Only used when hand:=true -->
+    <!-- Positional offset between $(arg arm_id)_hand -> $(arg arm_id)_hand_tcp [m]. Only used when hand:=true -->
     <xacro:arg name="tcp_xyz" default="0 0 0.1034" />
-    <!-- Rotational offset between $(arm_id)_hand -> $(arm_id)_hand_tcp [rad]. Only used when hand:=true -->
+    <!-- Rotational offset between $(arg arm_id)_hand -> $(arg arm_id)_hand_tcp [rad]. Only used when hand:=true -->
     <xacro:arg name="tcp_rpy" default="0 0 0" />
     <!-- Is the robot being simulated in gazebo?" -->
@@ -14,27 +14,36 @@
     <xacro:include filename="$(find franka_description)/robots/common/franka_arm.xacro" />
     <xacro:include filename="$(find softhands_description)/urdf/softhands.xacro"/>
-    <xacro:franka_arm arm_id="${arm_id}" safety_distance="0.03" gazebo="$(arg gazebo)" joint_limits="${joint_limits}"/>
+    <xacro:franka_arm arm_id="$(arg arm_id)" safety_distance="0.03" gazebo="$(arg gazebo)" joint_limits="${joint_limits}"/>
     <xacro:if value="$(arg hand)">
-	<!-- HAND LINK -->
-	<joint name="right_hand_ee_joint" type="fixed">
-		<origin xyz="0.130 0.000 0.035" rpy="0 0 0"/>
-		<parent link="${arm_id}_link8" />
-		<child link="right_hand_ee_link" />
-	</joint>
-	<link name="right_hand_ee_link">
-	</link>
-	<!-- RIGHT SOFTHAND -->
-	<!-- <xacro:flange_macro parent="${arm_id}_link8" name="flange">
-		<origin rpy="0 0 0" xyz="0 0 0.04"/>
-	</xacro:flange_macro> -->
-	<xacro:softhands type="right"
-		version = "v1.0_simple"
-		parent = "${arm_id}_link8"
-		position ="0.05 -0.00 0.04"
-		orientation ="0 -1.57 3.14"
-		operation_mode = "0"
-		translation="0.0">
-	</xacro:softhands>
-	    </xacro:if>
+		<xacro:include filename="$(find softhands_description)/urdf/xacro/include/macro/v1_2_research/header.xacro"/>
+		<xacro:include filename="$(find softhands_description)/urdf/xacro/v1_2_research.xacro"/>
+		<!-- HAND LINK -->
+		<joint name="right_hand_ee_joint" type="fixed">
+			<origin xyz="0.130 0.000 0.035" rpy="0 0 0"/>
+			<parent link="$(arg arm_id)_link8" />
+			<child link="right_hand_ee_link" />
+		</joint>
+		<link name="right_hand_ee_link">
+		</link>
+		<!-- RIGHT SOFTHAND -->
+		<!-- <xacro:flange_macro parent="$(arg arm_id)_link8" name="flange">
+			<origin rpy="0 0 0" xyz="0 0 0.04"/>
+		</xacro:flange_macro> -->
+		<!-- <xacro:softhands type="right"
+			version = "v1.0_simple"
+			parent = "$(arg arm_id)_link8"
+			position ="0.05 -0.00 0.04"
+			orientation ="0 -1.57 3.14"
+			operation_mode = "0"
+			translation="0.0">
+		</xacro:softhands> -->
+		<xacro:v1_2_research
+			side = "right"
+			parent = "$(arg arm_id)_link8"
+			position ="0 0 0"
+			orientation ="0 0 0"
+			fixed_hands="false">
+		</xacro:v1_2_research>
+	</xacro:if>
     <!-- Define additional Gazebo tags -->
     <xacro:if value="$(arg gazebo)">
@@ -48,29 +57,29 @@
         <child  link="$(arg arm_id)_link0" />
       </joint>
-      <xacro:gazebo-joint joint="${arm_id}_joint1" transmission="hardware_interface/PositionJointInterface" />
-      <xacro:gazebo-joint joint="${arm_id}_joint2" transmission="hardware_interface/PositionJointInterface" />
-      <xacro:gazebo-joint joint="${arm_id}_joint3" transmission="hardware_interface/PositionJointInterface" />
-      <xacro:gazebo-joint joint="${arm_id}_joint4" transmission="hardware_interface/PositionJointInterface" />
-      <xacro:gazebo-joint joint="${arm_id}_joint5" transmission="hardware_interface/PositionJointInterface" />
-      <xacro:gazebo-joint joint="${arm_id}_joint6" transmission="hardware_interface/PositionJointInterface" />
-      <xacro:gazebo-joint joint="${arm_id}_joint7" transmission="hardware_interface/PositionJointInterface" />
-      <xacro:gazebo-joint joint="${arm_id}_joint1" transmission="hardware_interface/VelocityJointInterface" />
-      <xacro:gazebo-joint joint="${arm_id}_joint2" transmission="hardware_interface/VelocityJointInterface" />
-      <xacro:gazebo-joint joint="${arm_id}_joint3" transmission="hardware_interface/VelocityJointInterface" />
-      <xacro:gazebo-joint joint="${arm_id}_joint4" transmission="hardware_interface/VelocityJointInterface" />
-      <xacro:gazebo-joint joint="${arm_id}_joint5" transmission="hardware_interface/VelocityJointInterface" />
-      <xacro:gazebo-joint joint="${arm_id}_joint6" transmission="hardware_interface/VelocityJointInterface" />
-      <xacro:gazebo-joint joint="${arm_id}_joint7" transmission="hardware_interface/VelocityJointInterface" />
-      <xacro:gazebo-joint joint="${arm_id}_joint1" transmission="hardware_interface/EffortJointInterface" />
-      <xacro:gazebo-joint joint="${arm_id}_joint2" transmission="hardware_interface/EffortJointInterface" />
-      <xacro:gazebo-joint joint="${arm_id}_joint3" transmission="hardware_interface/EffortJointInterface" />
-      <xacro:gazebo-joint joint="${arm_id}_joint4" transmission="hardware_interface/EffortJointInterface" />
-      <xacro:gazebo-joint joint="${arm_id}_joint5" transmission="hardware_interface/EffortJointInterface" />
-      <xacro:gazebo-joint joint="${arm_id}_joint6" transmission="hardware_interface/EffortJointInterface" />
-      <xacro:gazebo-joint joint="${arm_id}_joint7" transmission="hardware_interface/EffortJointInterface" />
-      <xacro:transmission-franka-state arm_id="${arm_id}" />
-      <xacro:transmission-franka-model arm_id="${arm_id}"
-         root="${arm_id}_joint1"
-         tip="${arm_id}_joint8"
+      <xacro:gazebo-joint joint="$(arg arm_id)_joint1" transmission="hardware_interface/PositionJointInterface" />
+      <xacro:gazebo-joint joint="$(arg arm_id)_joint2" transmission="hardware_interface/PositionJointInterface" />
+      <xacro:gazebo-joint joint="$(arg arm_id)_joint3" transmission="hardware_interface/PositionJointInterface" />
+      <xacro:gazebo-joint joint="$(arg arm_id)_joint4" transmission="hardware_interface/PositionJointInterface" />
+      <xacro:gazebo-joint joint="$(arg arm_id)_joint5" transmission="hardware_interface/PositionJointInterface" />
+      <xacro:gazebo-joint joint="$(arg arm_id)_joint6" transmission="hardware_interface/PositionJointInterface" />
+      <xacro:gazebo-joint joint="$(arg arm_id)_joint7" transmission="hardware_interface/PositionJointInterface" />
+      <xacro:gazebo-joint joint="$(arg arm_id)_joint1" transmission="hardware_interface/VelocityJointInterface" />
+      <xacro:gazebo-joint joint="$(arg arm_id)_joint2" transmission="hardware_interface/VelocityJointInterface" />
+      <xacro:gazebo-joint joint="$(arg arm_id)_joint3" transmission="hardware_interface/VelocityJointInterface" />
+      <xacro:gazebo-joint joint="$(arg arm_id)_joint4" transmission="hardware_interface/VelocityJointInterface" />
+      <xacro:gazebo-joint joint="$(arg arm_id)_joint5" transmission="hardware_interface/VelocityJointInterface" />
+      <xacro:gazebo-joint joint="$(arg arm_id)_joint6" transmission="hardware_interface/VelocityJointInterface" />
+      <xacro:gazebo-joint joint="$(arg arm_id)_joint7" transmission="hardware_interface/VelocityJointInterface" />
+      <xacro:gazebo-joint joint="$(arg arm_id)_joint1" transmission="hardware_interface/EffortJointInterface" />
+      <xacro:gazebo-joint joint="$(arg arm_id)_joint2" transmission="hardware_interface/EffortJointInterface" />
+      <xacro:gazebo-joint joint="$(arg arm_id)_joint3" transmission="hardware_interface/EffortJointInterface" />
+      <xacro:gazebo-joint joint="$(arg arm_id)_joint4" transmission="hardware_interface/EffortJointInterface" />
+      <xacro:gazebo-joint joint="$(arg arm_id)_joint5" transmission="hardware_interface/EffortJointInterface" />
+      <xacro:gazebo-joint joint="$(arg arm_id)_joint6" transmission="hardware_interface/EffortJointInterface" />
+      <xacro:gazebo-joint joint="$(arg arm_id)_joint7" transmission="hardware_interface/EffortJointInterface" />
+      <xacro:transmission-franka-state arm_id="$(arg arm_id)" />
+      <xacro:transmission-franka-model arm_id="$(arg arm_id)"
+         root="$(arg arm_id)_joint1"
+         tip="$(arg arm_id)_joint8"
        />
       <gazebo>
